Commit message: quadruped

File: body.urdf (robot description, URDF)
Before this commit: robot robot, 3 links, 2 joints
Links:
- added link BackLowerLeg, mass 1; collision box size=0.2 0.2 1; visual box size=0.2 0.2 1
- added link FrontLowerLeg, mass 1; collision box size=0.2 0.2 1; visual box size=0.2 0.2 1
- added link LeftLeg, mass 1; collision box size=1 0.2 0.2; visual box size=1 0.2 0.2
- added link LeftLowerLeg, mass 1; collision box size=0.2 0.2 1; visual box size=0.2 0.2 1
- added link RightLeg, mass 1; collision box size=1 0.2 0.2; visual box size=1 0.2 0.2
- added link RightLowerLeg, mass 1; collision box size=0.2 0.2 1; visual box size=0.2 0.2 1
- link BackLeg: geometry collision box size=0.2 1 0.2; visual box size=0.2 1 0.2
- link FrontLeg: geometry collision box size=0.2 1 0.2; visual box size=0.2 1 0.2
Joints:
- added joint BackLeg_BackLowerLeg: type revolute, parent BackLeg, child BackLowerLeg, origin xyz=0 -1 0 rpy=0 0 0, axis 1 0 0, limit lower=-3.14159 upper=3.14159 effort=0.0 velocity=0.0
- added joint FrontLeg_FrontLowerLeg: type revolute, parent FrontLeg, child FrontLowerLeg, origin xyz=0 1 0 rpy=0 0 0, axis 1 0 0, limit lower=-3.14159 upper=3.14159 effort=0.0 velocity=0.0
- added joint LeftLeg_LeftLowerLeg: type revolute, parent LeftLeg, child LeftLowerLeg, origin xyz=-1 0 0 rpy=0 0 0, axis 0 1 0, limit lower=-3.14159 upper=3.14159 effort=0.0 velocity=0.0
- added joint RightLeg_RightLowerLeg: type revolute, parent RightLeg, child RightLowerLeg, origin xyz=1 0 0 rpy=0 0 0, axis 0 1 0, limit lower=-3.14159 upper=3.14159 effort=0.0 velocity=0.0
- added joint Torso_LeftLeg: type revolute, parent Torso, child LeftLeg, origin xyz=-0.5 0 1 rpy=0 0 0, axis 0 1 0, limit lower=-3.14159 upper=3.14159 effort=0.0 velocity=0.0
- added joint Torso_RightLeg: type revolute, parent Torso, child RightLeg, origin xyz=0.5 0 1 rpy=0 0 0, axis 0 1 0, limit lower=-3.14159 upper=3.14159 effort=0.0 velocity=0.0
- joint Torso_BackLeg: axis 0 1 0 -> 1 0 0; origin xyz=-0.5 0 1 rpy=0 0 0 -> xyz=0 -0.5 1 rpy=0 0 0
- joint Torso_FrontLeg: axis 0 1 0 -> 1 0 0; origin xyz=0.5 0 1 rpy=0 0 0 -> xyz=0 0.5 1 rpy=0 0 0

Commit message: final project

File: body.urdf (robot description, URDF)
Before this commit: robot robot, 9 links, 8 joints
Links:
- removed link BackLeg
- removed link BackLowerLeg
- removed link FrontLeg
- removed link FrontLowerLeg
- added link LeftAnkle, mass 1; collision box size=0.1 0.1 0.5; visual box size=0.1 0.1 0.5
- added link LeftArm, mass 1; collision box size=0.1 0.1 1; visual box size=0.1 0.1 1
- added link LeftUpperArm, mass 1; collision box size=0.1 0.1 1; visual box size=0.1 0.1 1
- added link LeftWrist, mass 1; collision box size=0.1 0.1 0.5; visual box size=0.1 0.1 0.5
- added link RightAnkle, mass 1; collision box size=0.1 0.1 0.5; visual box size=0.1 0.1 0.5
- added link RightArm, mass 1; collision box size=0.1 0.1 1; visual box size=0.1 0.1 1
- added link RightUpperArm, mass 1; collision box size=0.1 0.1 1; visual box size=0.1 0.1 1
- added link RightWrist, mass 1; collision box size=0.1 0.1 0.5; visual box size=0.1 0.1 0.5
- link LeftLeg: geometry collision box size=0.1 0.1 1; visual box size=0.1 0.1 1
- link LeftLowerLeg: geometry collision box size=0.1 0.1 1; visual box size=0.1 0.1 1
- link RightLeg: geometry collision box size=0.1 0.1 1; visual box size=0.1 0.1 1
- link RightLowerLeg: geometry collision box size=0.1 0.1 1; visual box size=0.1 0.1 1
- link Torso: geometry collision box size=0.5 1 1; visual box size=0.5 1 1
Joints:
- removed joint BackLeg_BackLowerLeg
- removed joint FrontLeg_FrontLowerLeg
- removed joint Torso_BackLeg
- removed joint Torso_FrontLeg
- added joint LeftArm_LeftUpperArm: type revolute, parent LeftArm, child LeftUpperArm, origin xyz=0 0 1 rpy=0 0 0, axis 0 1 0, limit lower=-3.14159 upper=3.14159 effort=0.0 velocity=0.0
- added joint LeftLowerLeg_LeftAnkle: type revolute, parent LeftLowerLeg, child LeftAnkle, origin xyz=0 0 -1 rpy=0 0 0, axis 0 1 0, limit lower=-3.14159 upper=3.14159 effort=0.0 velocity=0.0
- added joint LeftUpperArm_LeftWrist: type revolute, parent LeftUpperArm, child LeftWrist, origin xyz=0 0 1 rpy=0 0 0, axis 0 1 0, limit lower=-3.14159 upper=3.14159 effort=0.0 velocity=0.0
- added joint RightArm_RightUpperArm: type revolute, parent RightArm, child RightUpperArm, origin xyz=0 0 1 rpy=0 0 0, axis 0 1 0, limit lower=-3.14159 upper=3.14159 effort=0.0 velocity=0.0
- added joint RightLowerLeg_RightAnkle: type revolute, parent RightLowerLeg, child RightAnkle, origin xyz=0 0 -1 rpy=0 0 0, axis 0 1 0, limit lower=-3.14159 upper=3.14159 effort=0.0 velocity=0.0
- added joint RightUpperArm_RightWrist: type revolute, parent RightUpperArm, child RightWrist, origin xyz=0 0 1 rpy=0 0 0, axis 0 1 0, limit lower=-3.14159 upper=3.14159 effort=0.0 velocity=0.0
- added joint Torso_LeftArm: type revolute, parent Torso, child LeftArm, origin xyz=0 -0.5 0.5 rpy=0 0 0, axis 0 1 0, limit lower=-3.14159 upper=3.14159 effort=0.0 velocity=0.0
- added joint Torso_RightArm: type revolute, parent Torso, child RightArm, origin xyz=0 0.5 0.5 rpy=0 0 0, axis 0 1 0, limit lower=-3.14159 upper=3.14159 effort=0.0 velocity=0.0
- joint LeftLeg_LeftLowerLeg: origin xyz=-1 0 0 rpy=0 0 0 -> xyz=0 0 -1 rpy=0 0 0
- joint RightLeg_RightLowerLeg: origin xyz=1 0 0 rpy=0 0 0 -> xyz=0 0 -1 rpy=0 0 0
- joint Torso_LeftLeg: origin xyz=-0.5 0 1 rpy=0 0 0 -> xyz=0 -0.5 0 rpy=0 0 0
- joint Torso_RightLeg: origin xyz=0.5 0 1 rpy=0 0 0 -> xyz=0 0.5 0 rpy=0 0 0

Commit message: yes

File: body.urdf (robot description, URDF)
Before this commit: robot robot, 13 links, 12 joints
Links:
- removed link LeftAnkle
- removed link LeftArm
- removed link LeftLeg
- removed link LeftLowerLeg
- removed link LeftUpperArm
- removed link LeftWrist
- removed link RightAnkle
- removed link RightArm
- removed link RightLeg
- removed link RightLowerLeg
- removed link RightUpperArm
- removed link RightWrist
- removed link Torso
- added link Link0, mass 1; collision box size=0.771000158042149 0.8360523204494051 0.23575925266138442; visual box size=0.771000158042149 0.8360523204494051 0.23575925266138442
- added link Link1, mass 1; collision box size=0.7514275870640137 0.13079464112806927 0.8163618805789009; visual box size=0.7514275870640137 0.13079464112806927 0.8163618805789009
- added link Link2, mass 1; collision box size=0.27227126880036434 0.8461951499636334 0.8302972565996962; visual box size=0.27227126880036434 0.8461951499636334 0.8302972565996962
- added link Link3, mass 1; collision box size=0.7697656438209526 0.05217759513577602 0.8882971951292685; visual box size=0.7697656438209526 0.05217759513577602 0.8882971951292685
- added link Link4, mass 1; collision box size=0.6525470912962759 0.7360569453142063 0.47497572318445613; visual box size=0.6525470912962759 0.7360569453142063 0.47497572318445613
- added link Link5, mass 1; collision box size=0.007120423660419317 0.9147285529275258 0.9778201187517719; visual box size=0.007120423660419317 0.9147285529275258 0.9778201187517719
- added link Link6, mass 1; collision box size=0.7690075913992069 0.8991928974260932 0.36798947783011204; visual box size=0.7690075913992069 0.8991928974260932 0.36798947783011204
- added link Link7, mass 1; collision box size=0.7255275785606176 0.4437258681329107 0.9179498550577707; visual box size=0.7255275785606176 0.4437258681329107 0.9179498550577707
Joints:
- removed joint LeftArm_LeftUpperArm
- removed joint LeftLeg_LeftLowerLeg
- removed joint LeftLowerLeg_LeftAnkle
- removed joint LeftUpperArm_LeftWrist
- removed joint RightArm_RightUpperArm
- removed joint RightLeg_RightLowerLeg
- removed joint RightLowerLeg_RightAnkle
- removed joint RightUpperArm_RightWrist
- removed joint Torso_LeftArm
- removed joint Torso_LeftLeg
- removed joint Torso_RightArm
- removed joint Torso_RightLeg
- added joint Link0_Link1: type revolute, parent Link0, child Link1, origin xyz=0.3855000790210745 0 0.48891005937588594 rpy=0 0 0, axis 1 0 0, limit lower=-3.14159 upper=3.14159 effort=0.0 velocity=0.0
- added joint Link1_Link2: type revolute, parent Link1, child Link2, origin xyz=0.7514275870640137 0 0 rpy=0 0 0, axis 1 0 0, limit lower=-3.14159 upper=3.14159 effort=0.0 velocity=0.0
- added joint Link2_Link3: type revolute, parent Link2, child Link3, origin xyz=0.27227126880036434 0 0 rpy=0 0 0, axis 0 1 0, limit lower=-3.14159 upper=3.14159 effort=0.0 velocity=0.0
- added joint Link3_Link4: type revolute, parent Link3, child Link4, origin xyz=0.7697656438209526 0 0 rpy=0 0 0, axis 1 0 0, limit lower=-3.14159 upper=3.14159 effort=0.0 velocity=0.0
- added joint Link4_Link5: type revolute, parent Link4, child Link5, origin xyz=0.6525470912962759 0 0 rpy=0 0 0, axis 0 0 1, limit lower=-3.14159 upper=3.14159 effort=0.0 velocity=0.0
- added joint Link5_Link6: type revolute, parent Link5, child Link6, origin xyz=0.007120423660419317 0 0 rpy=0 0 0, axis 0 0 1, limit lower=-3.14159 upper=3.14159 effort=0.0 velocity=0.0
- added joint Link6_Link7: type revolute, parent Link6, child Link7, origin xyz=0.7690075913992069 0 0 rpy=0 0 0, axis 0 0 1, limit lower=-3.14159 upper=3.14159 effort=0.0 velocity=0.0

Commit message: ye

File: body.urdf (robot description, URDF)
Before this commit: robot robot, 8 links, 7 joints
Links:
- added link Link8, mass 1; collision box size=0.34549244817673797 0.6845930236184958 0.8703845964585442; visual box size=0.34549244817673797 0.6845930236184958 0.8703845964585442
- link Link0: geometry collision box size=0.7070208138297192 0.27074402265736464 0.3776333168041439; visual box size=0.7070208138297192 0.27074402265736464 0.3776333168041439
- link Link1: geometry collision box size=0.894857903615321 0.5941842535780172 0.24702289748178285; visual box size=0.894857903615321 0.5941842535780172 0.24702289748178285
- link Link2: geometry collision box size=0.14096690820783808 0.8175005605504191 0.5062471042108229; visual box size=0.14096690820783808 0.8175005605504191 0.5062471042108229
- link Link3: geometry collision box size=0.21122499308023646 0.6086642536681557 0.9232636889391284; visual box size=0.21122499308023646 0.6086642536681557 0.9232636889391284
- link Link4: geometry collision box size=0.14149911656819059 0.39074939166886047 0.9117346004894938; visual box size=0.14149911656819059 0.39074939166886047 0.9117346004894938
- link Link5: geometry collision box size=0.2623013315313367 0.6061194138184565 0.16126972346863722; visual box size=0.2623013315313367 0.6061194138184565 0.16126972346863722
- link Link6: geometry collision box size=0.9937803613290258 0.38099819693326165 0.6828256440012921; visual box size=0.9937803613290258 0.38099819693326165 0.6828256440012921
- link Link7: geometry collision box size=0.2014746105743298 0.5488253621671542 0.6621933401960012; visual box size=0.2014746105743298 0.5488253621671542 0.6621933401960012
Joints:
- added joint Link7_Link8: type revolute, parent Link7, child Link8, origin xyz=0.2014746105743298 0 0 rpy=0 0 0, axis 1 0 0, limit lower=-3.14159 upper=3.14159 effort=0.0 velocity=0.0
- joint Link0_Link1: origin xyz=0.3855000790210745 0 0.48891005937588594 rpy=0 0 0 -> xyz=0.3535104069148596 0 0.4616318444695642 rpy=0 0 0
- joint Link1_Link2: origin xyz=0.7514275870640137 0 0 rpy=0 0 0 -> xyz=0.894857903615321 0 0 rpy=0 0 0
- joint Link2_Link3: origin xyz=0.27227126880036434 0 0 rpy=0 0 0 -> xyz=0.14096690820783808 0 0 rpy=0 0 0
- joint Link3_Link4: axis 1 0 0 -> 0 1 0; origin xyz=0.7697656438209526 0 0 rpy=0 0 0 -> xyz=0.21122499308023646 0 0 rpy=0 0 0
- joint Link4_Link5: axis 0 0 1 -> 1 0 0; origin xyz=0.6525470912962759 0 0 rpy=0 0 0 -> xyz=0.14149911656819059 0 0 rpy=0 0 0
- joint Link5_Link6: origin xyz=0.007120423660419317 0 0 rpy=0 0 0 -> xyz=0.2623013315313367 0 0 rpy=0 0 0
- joint Link6_Link7: origin xyz=0.7690075913992069 0 0 rpy=0 0 0 -> xyz=0.9937803613290258 0 0 rpy=0 0 0

Commit message: te

File: body.urdf (robot description, URDF)
Before this commit: robot robot, 9 links, 8 joints
Links:
- removed link Link5
- removed link Link6
- removed link Link7
- removed link Link8
- link Link0: geometry collision box size=0.3872675945979489 0.7930130119237252 0.3219849786517617; visual box size=0.3872675945979489 0.7930130119237252 0.3219849786517617
- link Link1: geometry collision box size=0.9297432945132085 0.049076668974213145 0.3487241274256687; visual box size=0.9297432945132085 0.049076668974213145 0.3487241274256687
- link Link2: geometry collision box size=0.643233346092724 0.40285904268594874 0.027054731037775448; visual box size=0.643233346092724 0.40285904268594874 0.027054731037775448
- link Link3: geometry collision box size=0.2314134144773835 0.03212634234273026 0.41801029439377835; visual box size=0.2314134144773835 0.03212634234273026 0.41801029439377835
- link Link4: geometry collision box size=0.167759182808203 0.2506867943689979 0.06870749578287483; visual box size=0.167759182808203 0.2506867943689979 0.06870749578287483
Joints:
- removed joint Link1_Link2
- removed joint Link2_Link3
- removed joint Link3_Link4
- removed joint Link4_Link5
- removed joint Link5_Link6
- removed joint Link6_Link7
- removed joint Link7_Link8
- added joint Link0_Link2: type revolute, parent Link0, child Link2, origin xyz=-0.1452738487759643 0.3965065059618626 0.4515190972661096 rpy=0 0 0, axis 0 1 0, limit lower=-3.14159 upper=3.14159 effort=0.0 velocity=0.0
- added joint Link0_Link3: type revolute, parent Link0, child Link3, origin xyz=0.19363379729897445 0.29686132986118746 0.4650718227462075 rpy=0 0 0, axis 0 1 0, limit lower=-3.14159 upper=3.14159 effort=0.0 velocity=0.0
- added joint Link0_Link4: type revolute, parent Link0, child Link4, origin xyz=-0.06797560536202223 0.23931295272657804 0.6063387265431991 rpy=0 0 0, axis 1 0 0, limit lower=-3.14159 upper=3.14159 effort=0.0 velocity=0.0
- joint Link0_Link1: origin xyz=0.3535104069148596 0 0.4616318444695642 rpy=0 0 0 -> xyz=-0.19363379729897445 0.08095829896465795 0.5146197290351409 rpy=0 0 0
