Commit message: files

File: body0.urdf (robot description, URDF)
Before this commit: robot robot, 4 links, 3 joints
Links:
- added link Link4, mass 1; collision box size=0.3305446319587937 0.09092092241021377 0.9354705111785977; visual box size=0.3305446319587937 0.09092092241021377 0.9354705111785977
- link Link0: geometry collision box size=0.23034905261871041 0.941383796303741 0.9317065228160369; visual box size=0.23034905261871041 0.941383796303741 0.9317065228160369
- link Link1: geometry collision box size=0.5713845584914515 0.4247039685663452 0.5659332657487284; visual box size=0.5713845584914515 0.4247039685663452 0.5659332657487284
- link Link2: geometry collision box size=0.12601804579300113 0.6509409851688401 0.7759674204130412; visual box size=0.12601804579300113 0.6509409851688401 0.7759674204130412
- link Link3: geometry collision box size=0.35041237835429606 0.5777480110644839 0.22060456799906802; visual box size=0.35041237835429606 0.5777480110644839 0.22060456799906802
Joints:
- removed joint Link0_Link2
- removed joint Link0_Link3
- added joint Link1_Link2: type revolute, parent Link1, child Link2, origin xyz=-0.05639677500430956 -0.15152497150675429 -0.2829666328743642 rpy=0 0 0, axis 1 0 0, limit lower=-3.14159 upper=3.14159 effort=0.0 velocity=0.0
- added joint Link2_Link3: type revolute, parent Link2, child Link3, origin xyz=0.049443104117976255 0.32547049258442007 -0.07821722675109827 rpy=0 0 0, axis 0 1 0, limit lower=-3.14159 upper=3.14159 effort=0.0 velocity=0.0
- added joint Link3_Link4: type revolute, parent Link3, child Link4, origin xyz=0.09303695513508692 0.5777480110644839 -0.08274001262964788 rpy=0 0 0, axis 1 0 0, limit lower=-3.14159 upper=3.14159 effort=0.0 velocity=0.0
- joint Link0_Link1: axis 1 0 0 -> 0 0 1; origin xyz=0.0477469539085148 -0.30458556243261437 3.099249444626399 rpy=0 0 0 -> xyz=-0.11517452630935521 -0.005727947305645714 3.6625001868756994 rpy=0 0 0
